File: hardware/basicsensormodule.kicad_pcb (KiCad board)
At the start: 2 copper layers, 247.1 x 121 mm, 212 parts, among them J1 Conn_01x04, J401 USART, J601 RJ45, J602 RJ45, U201 MCP2551-I/SN, U202 MCP2515-xSO, U401 ATMEGA328P-PU, U501 LM7805, Y201 16MHz, Y401 16MHz

Commit message: PCB atualizada com as mudanças do raspberry
Foram adicionadas as mudanças do conector do raspberry e retirado algumas coisas não necessárias.
Parts:
- removed the C102 at (237.5, 43.4)
- removed the C102 at (172.5, 43.4)
- removed the C102 at (107.5, 43.4)
- removed the C102 at (42.5, 43.4)
- removed the C201 at (235.0, 94.0)
- removed the C201 at (170.0, 94.0)
- removed the C201 at (105.0, 94.0)
- removed the C201 at (40.0, 94.0)
- removed the C202 at (177.6, 109.9)
- removed the C202 at (112.6, 109.9)
- removed the C202 at (47.6, 109.9)
- removed the C203 at (162.4, 100.1)
- removed the C203 at (97.4, 100.1)
- removed the C203 at (32.4, 100.1)
- removed the C204 at (164.5, 96.3)
- removed the C204 at (99.5, 96.3)
- removed the C204 at (34.5, 96.3)
- removed the C205 at (172.8, 119.8)
- removed the C205 at (107.8, 119.8)
- removed the C205 at (42.8, 119.8)
- removed the C401 at (181.1, 73.4)
- removed the C401 at (116.1, 73.4)
- removed the C401 at (51.1, 73.4)
- removed C402 (x4), C405 (x4), C406 (x4): 100nF, Capacitor_SMD:C_0805_2012Metric_Pad1.15x1.40mm_HandSolder
- removed C403 (x4), C404 (x4): 22pF, Capacitor_SMD:C_0805_2012Metric_Pad1.15x1.40mm_HandSolder
- removed the C501 at (193.1, 95.9)
- removed the C501 at (128.1, 95.9)
- removed the C501 at (63.1, 95.9)
- removed the C502 at (193.1, 92.1)
- removed the C502 at (128.1, 92.1)
- removed the C502 at (63.1, 92.1)
- removed the C503 at (186.5, 95.2)
- removed the C503 at (121.5, 95.2)
- removed the C503 at (56.5, 95.2)
- removed the C504 at (186.5, 92.1)
- removed the C504 at (121.5, 92.1)
- removed the C504 at (56.5, 92.1)
- removed the D201 at (181.1, 124.8)
- removed the D201 at (116.1, 124.8)
- removed the D201 at (51.1, 124.8)
- removed D401 (x4): LL4148, Diode_SMD:D_MiniMELF_Handsoldering
- removed the D402 at (159.5, 88.4)
- removed the D402 at (94.5, 88.4)
- removed the D402 at (29.5, 88.4)
- removed the D403 at (159.5, 85.8)
- removed the D403 at (94.5, 85.8)
- removed the D403 at (29.5, 85.8)
- removed the D501 at (198.6, 109.2)
- removed the D501 at (133.6, 109.2)
- removed the D501 at (68.6, 109.2)
- removed the F501 at (198.6, 100.3)
- removed the F501 at (133.6, 100.3)
- removed the F501 at (68.6, 100.3)
- removed the H101 at (157.9, 38.1)
- removed the H101 at (92.9, 38.1)
- removed the H101 at (27.9, 38.1)
- removed the H102 at (221.9, 122.9)
- removed the H102 at (156.9, 122.9)
- removed the H102 at (91.9, 122.9)
- removed the H102 at (26.9, 122.9)
- removed the H103 at (200.1, 122.9)
- removed the H103 at (135.1, 122.9)
- removed the H103 at (70.1, 122.9)
- removed the H104 at (199.8, 38.1)
- removed the H104 at (134.8, 38.1)
- removed the H104 at (69.8, 38.1)
- removed the J1 at (244.5, 38.1)
- removed the J1 at (179.5, 38.1)
- removed the J1 at (114.5, 38.1)
- removed the J1 at (49.5, 38.1)
- removed the J401 at (156.9, 60.7)
- removed the J401 at (91.9, 60.7)
- removed the J401 at (26.9, 60.7)
- removed the J601 at (183.6, 135.6)
- removed the J601 at (118.6, 135.6)
- removed the J601 at (53.6, 135.6)
- removed the J602 at (162.7, 135.6)
- removed the J602 at (97.7, 135.6)
- removed the J602 at (32.7, 135.6)
- removed the R201 at (181.1, 120.8)
- removed the R201 at (116.1, 120.8)
- removed the R201 at (51.1, 120.8)
- removed the R202 at (172.8, 121.9)
- removed the R202 at (107.8, 121.9)
- removed the R202 at (42.8, 121.9)
- removed the R203 at (181.0, 108.0)
- removed the R203 at (116.0, 108.0)
- removed the R203 at (51.0, 108.0)
- removed R401 (x4): 10k, Resistor_SMD:R_0805_2012Metric_Pad1.15x1.40mm_HandSolder
- removed the R402 at (229.5, 55.6)
- removed the R402 at (164.5, 55.6)
- removed the R402 at (99.5, 55.6)
- removed the R402 at (34.5, 55.6)
- removed the R403 at (164.5, 58.2)
- removed the R403 at (99.5, 58.2)
- removed the R403 at (34.5, 58.2)
- removed the R404 at (163.3, 88.4)
- removed the R404 at (98.3, 88.4)
- removed the R404 at (33.3, 88.4)
- removed the R405 at (163.3, 85.8)
- removed the R405 at (98.3, 85.8)
- removed the R405 at (33.3, 85.8)
- removed TP201 (x4): SI, TestPoint:TestPoint_Pad_2.0x2.0mm
- removed TP202 (x4): SO, TestPoint:TestPoint_Pad_2.0x2.0mm
- removed TP203 (x4): TXCAN, TestPoint:TestPoint_Pad_2.0x2.0mm
- removed TP204 (x4): RXCAN, TestPoint:TestPoint_Pad_2.0x2.0mm
- removed TP205 (x4): SC, TestPoint:TestPoint_Pad_2.0x2.0mm
- removed TP206 (x4): SCK, TestPoint:TestPoint_Pad_2.0x2.0mm
- removed TP207 (x4): CAN_H, TestPoint:TestPoint_Pad_2.0x2.0mm
- removed TP208 (x4): CAN_L, TestPoint:TestPoint_Pad_2.0x2.0mm
- removed TP209 (x4): INT, TestPoint:TestPoint_Pad_2.0x2.0mm
- removed the U201 at (172.8, 114.7)
- removed the U201 at (107.8, 114.7)
- removed the U201 at (42.8, 114.7)
- removed the U202 at (172.8, 102.6)
- removed the U202 at (107.8, 102.6)
- removed the U202 at (42.8, 102.6)
- removed U401 (x4): ATMEGA328P-PU, Package_DIP:DIP-28_W7.62mm_Socket
- removed the U501 at (257.2, 86.4)
- removed the U501 at (192.2, 86.4)
- removed the U501 at (127.2, 86.4)
- removed the U501 at (62.2, 86.4)
- removed the Y201 at (162.0, 102.6)
- removed the Y201 at (97.0, 102.6)
- removed the Y201 at (32.0, 102.6)
- removed Y401 (x4): 16MHz, Crystal:Crystal_HC49-U_Vertical
- added C102: 100nF, Capacitor_SMD:C_0805_2012Metric_Pad1.15x1.40mm_HandSolder, B.Cu at (241.3, 43.2)
- added C201: 100nF, Capacitor_SMD:C_0805_2012Metric_Pad1.15x1.40mm_HandSolder, B.Cu at (242.6, 109.9)
- added H102: MountingHole, MountingHole:MountingHole_3.2mm_M3, F.Cu at (221.0, 147.3)
- added J1: Conn_01x04, Connector_PinHeader_2.54mm:PinHeader_1x04_P2.54mm_Vertical, F.Cu at (230.5, 38.7)
- added J501: Raspberry_Pi_2_3, Connector_PinHeader_2.54mm:PinHeader_2x20_P2.54mm_Vertical, F.Cu at (259.7, 54.6)
- added R204: 22K, Resistor_SMD:R_0805_2012Metric_Pad1.15x1.40mm_HandSolder, B.Cu at (229.9, 109.9)
- added R205: 10K, Resistor_SMD:R_0805_2012Metric_Pad1.15x1.40mm_HandSolder, B.Cu at (234.3, 111.4)
- added R402: 1k, Resistor_SMD:R_0805_2012Metric_Pad1.15x1.40mm_HandSolder, B.Cu at (261.2, 43.4)
- added U501: LM7805, KicadZeniteSolarLibrary18:TO-220-3_Horizontal_TabDown_SMD, B.Cu at (228.3, 79.4)
- moved D501 46.3 mm to (221.0, 127.4)
- moved F501 45.7 mm to (221.0, 83.8)
- moved H104 43.9 mm to (221.0, 35.6)
- moved H101 42.6 mm to (265.4, 35.6)
- moved D402 40.7 mm to (256.6, 113.4), turned to 90 degrees
- moved D403 40.5 mm to (254.1, 113.4), turned to 90 degrees
- moved C503 37.4 mm to (223.5, 70.5), turned to 180 degrees
- moved J401 36.3 mm to (250.8, 38.7), turned to 90 degrees
- moved R404 35.4 mm to (256.6, 109.5), turned to 270 degrees
- moved C504 35.1 mm to (227.3, 66.7)
- moved R405 35.1 mm to (254.1, 109.5), turned to 270 degrees
- moved C502 34.0 mm to (224.8, 85.1), turned to 270 degrees
- moved R403 34.0 mm to (261.2, 45.7)
- moved C501 30.0 mm to (229.2, 87.6), turned to 270 degrees
- moved C401 26.4 mm to (257.4, 49.5)
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Connections:
- C205 pad 1: +5V -> /CANBUS/3V3
- J401 pad 4: Net-(C405-Pad2) -> (no net)
- R203 pad 1: +5V -> /CANBUS/3V3
- U201 pad 4: /CANBUS/RXCAN -> Net-(R205-Pad1)
- U201 pad 5: Net-(U201-Pad5) -> (no net)
- U202 pad 10: Net-(U202-Pad10) -> (no net)
- U202 pad 11: Net-(U202-Pad11) -> (no net)
- U202 pad 18: +5V -> /CANBUS/3V3
- U202 pad 3: Net-(U202-Pad3) -> (no net)
- U202 pad 4: Net-(U202-Pad4) -> (no net)
- U202 pad 5: Net-(U202-Pad5) -> (no net)
- U202 pad 6: Net-(U202-Pad6) -> (no net)
Routing:
- net +5V: track 807.1 -> 168.3 mm
- net GND: track 318.1 -> 39.4 mm, vias 56 -> 5
- net /POWER SUPPLY/+18V_IN: track 287.8 -> 73.5 mm
- net /CANBUS CONN/CAN_H: track 202.3 -> 48.6 mm
- net /CANBUS CONN/CAN_L: track 192.7 -> 45.4 mm, vias 8 -> 2
- net /MISO: track 150.9 -> 34.0 mm, vias 0 -> 2
- net /SCK: track 142.3 -> 30.2 mm
- net /CANBUS/3V3: track 0.00 -> 97.8 mm
- net /MOSI: track 131.5 -> 38.6 mm
- net /CANBUS/CS: track 128.6 -> 36.9 mm
- net /MCU/SDA: track 92.5 -> 35.8 mm
- net /MCU/RESET: track 49.5 -> 0.00 mm
- net /CANBUS/TXCAN: track 61.4 -> 13.9 mm
- net /CANBUS/INT: track 84.4 -> 37.6 mm, vias 0 -> 2
- net /CANBUS/RXCAN: track 56.5 -> 11.2 mm
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Other:
- board size 247.1 x 121 mm -> 52.1 x 121 mm

Commit message: Project cleaned
Parts:
- J1: value Conn_01x04 -> I2C
- moved H101 173.9 mm to (97.1, 79.1), turned to 0 degrees
- moved R402 161.3 mm to (104.9, 83.3), turned to 270 degrees
- moved J401 160.3 mm to (100.2, 93.7), turned to 180 degrees
- moved R403 158.5 mm to (107.2, 83.3), turned to 270 degrees
- moved H104 152.0 mm to (97.1, 123.5), turned to 0 degrees
- moved C401 151.1 mm to (111.0, 87.1), turned to 90 degrees
- moved J1 150.4 mm to (100.2, 114.0), turned to 180 degrees
- moved C102 149.2 mm to (104.7, 103.2), turned to 90 degrees
- moved J501 146.7 mm to (116.1, 84.8), turned to 90 degrees
- moved C504 111.3 mm to (128.2, 117.2), turned to 90 degrees
- moved C503 104.5 mm to (132.0, 121.0), turned to 270 degrees
- moved U501 94.9 mm to (140.9, 116.2), turned to 180 degrees
- moved H103 88.7 mm to (208.8, 79.1), turned to 0 degrees
- moved R404 88.3 mm to (171.0, 87.9), turned to 0 degrees
- moved D402 85.7 mm to (174.9, 87.9), turned to 180 degrees
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Routing:
- net (no net): vias 0 -> 1
Other:
- board size 52.1 x 121 mm -> 121 x 52.1 mm
- board text added: "+3V3"
- board text added: "GND"
- board text added: "RXD/GPIO10 (pin 10)"
- board text added: "SCL/GPIO03 (pin 5)"
- board text added: "SDA/GPIO02 (pin 3)"
- board text added: "TXD/GPIO14 (pin 8)"
