File: hardware/canbus.sch (KiCad schematic (older format))
At the start: 21 parts, among them U201 MCP2551-I/SN, U202 MCP2515-xSO, Y201 16MHz

Commit message: Adicão da alimentação de uma folha para outra .
Alimentação de 3V3.
Parts:
- added R204: 22K, symbol Device:R_Small
- added R205: 10K, symbol Device:R_Small
Connections:
- net labels added: 3V3
- wire segments 86 -> 89
Other:
- moved on the sheet: C201, C203, C204, C205, R203, U202, Y201

Commit message: PCB atualizada com as mudanças do raspberry
Foram adicionadas as mudanças do conector do raspberry e retirado algumas coisas não necessárias.
Parts:
- R204, R205: footprint (none) -> Resistor_SMD:R_0805_2012Metric_Pad1.15x1.40mm_HandSolder
Connections:
- wire segments 89 -> 88
Other:
- moved on the sheet: R204, R205
Changed lines of the file:
@@
 $EndComp
 Wire Wire Line
-	4250 3100 4600 3100
-Wire Wire Line
-	4250 3200 5950 3200
+	4250 3200 4600 3200
 Wire Wire Line
 	3700 3700 3800 3700
@@
 	2300 4100 2400 4100
 $Comp
-L power:+5V #PWR0107
-U 1 1 5BEBB382
-P 4250 4150
-F 0 "#PWR0107" H 4250 4000 50  0001 C CNN
-F 1 "+5V" H 4300 4350 50  0000 C CNN
-F 2 "" H 4250 4150 50  0001 C CNN
-F 3 "" H 4250 4150 50  0001 C CNN
-	1    4250 4150
-	1    0    0    -1
-$EndComp
-Wire Wire Line
-	4250 4150 4250 4300
-Connection ~ 4250 4300
-$Comp
 L basicsensormodule-rescue:MCP2515-xSO-Interface_CAN_LIN U202
 U 1 1 5BE69763
@@
 L Device:R_Small R205
 U 1 1 5CD56C8C
-P 4850 3100
-F 0 "R205" V 4654 3100 50  0000 C CNN
-F 1 "10K" V 4745 3100 50  0000 C CNN
-F 2 "" H 4850 3100 50  0001 C CNN
-F 3 "~" H 4850 3100 50  0001 C CNN
-	1    4850 3100
+P 4850 3200
+F 0 "R205" V 4654 3200 50  0000 C CNN
+F 1 "10K" V 4745 3200 50  0000 C CNN
+F 2 "Resistor_SMD:R_0805_2012Metric_Pad1.15x1.40mm_HandSolder" H 4850 3200 50  0001 C CNN
+F 3 "~" H 4850 3200 50  0001 C CNN
+	1    4850 3200
 	0    1    1    0
 $EndComp
@@
 L Device:R_Small R204
 U 1 1 5CD57829
-P 4600 3200
-F 0 "R204" H 4541 3154 50  0000 R CNN
-F 1 "22K" H 4541 3245 50  0000 R CNN
-F 2 "" H 4600 3200 50  0001 C CNN
-F 3 "~" H 4600 3200 50  0001 C CNN
-	1    4600 3200
+P 4600 3300
+F 0 "R204" H 4541 3254 50  0000 R CNN
+F 1 "22K" H 4541 3345 50  0000 R CNN
+F 2 "Resistor_SMD:R_0805_2012Metric_Pad1.15x1.40mm_HandSolder" H 4600 3300 50  0001 C CNN
+F 3 "~" H 4600 3300 50  0001 C CNN
+	1    4600 3300
 	-1   0    0    1
 $EndComp
-Connection ~ 4600 3100
-Wire Wire Line
-	4600 3100 4750 3100
-Wire Wire Line
-	4950 3100 5950 3100
 $Comp
 L power:GND #PWR0201
 U 1 1 5CD5B5AA
-P 4600 3450
-F 0 "#PWR0201" H 4600 3200 50  0001 C CNN
-F 1 "GND" H 4605 3277 50  0000 C CNN
-F 2 "" H 4600 3450 50  0001 C CNN
-F 3 "" H 4600 3450 50  0001 C CNN
-	1    4600 3450
-	1    0    0    -1
-$EndComp
-Wire Wire Line
-	4600 3300 4600 3450
+P 4600 3550
+F 0 "#PWR0201" H 4600 3300 50  0001 C CNN
+F 1 "GND" H 4605 3377 50  0000 C CNN
+F 2 "" H 4600 3550 50  0001 C CNN
+F 3 "" H 4600 3550 50  0001 C CNN
+	1    4600 3550
+	1    0    0    -1
+$EndComp
+Wire Wire Line
+	4600 3400 4600 3550
+Text Label 3100 2350 0    50   ~ 0
+3V3
+Text Label 4250 4300 0    50   ~ 0
+3V3
+Connection ~ 4600 3200
+Wire Wire Line
+	4600 3200 4750 3200
+Wire Wire Line
+	4950 3200 5950 3200
+Wire Wire Line
+	4250 3100 5950 3100
 $EndSCHEMATC

Commit message: Project cleaned
Parts:
- TP201, TP202, TP203, TP204, TP205, TP206, TP207, TP208, TP209: symbol basicsensormodule-rescue:TestPoint-Connector -> Connector:TestPoint
Changed lines of the file:
@@
 EMI/ESD Protection Solutions for the CAN Bus: \nhttps://www.onsemi.com/pub/Collateral/AND8169-D.PDF\nSparkFun CAN-Bus Shield:\nhttps://cdn.sparkfun.com/datasheets/Dev/Arduino/Shields/SparkFun_CAN-Bus_Shield_v13a.pdf
 $Comp
-L basicsensormodule-rescue:TestPoint-Connector TP203
+L Connector:TestPoint TP203
 U 1 1 5AAC2327
 P 4250 3050
@@
 $EndComp
 $Comp
-L basicsensormodule-rescue:TestPoint-Connector TP204
+L Connector:TestPoint TP204
 U 1 1 5AAC23CC
 P 4250 3250
@@
 Connection ~ 4250 3200
 $Comp
-L basicsensormodule-rescue:TestPoint-Connector TP209
+L Connector:TestPoint TP209
 U 1 1 5AAC2B03
 P 3700 3650
@@
 $EndComp
 $Comp
-L basicsensormodule-rescue:TestPoint-Connector TP201
+L Connector:TestPoint TP201
 U 1 1 5AAC2C42
 P 2250 3000
@@
 $EndComp
 $Comp
-L basicsensormodule-rescue:TestPoint-Connector TP202
+L Connector:TestPoint TP202
 U 1 1 5AAC2C8C
 P 2100 3050
@@
 $EndComp
 $Comp
-L basicsensormodule-rescue:TestPoint-Connector TP206
+L Connector:TestPoint TP206
 U 1 1 5AAC2CDB
 P 1800 3550
@@
 $EndComp
 $Comp
-L basicsensormodule-rescue:TestPoint-Connector TP205
+L Connector:TestPoint TP205
 U 1 1 5AAC2E79
 P 1950 3450
@@
 Connection ~ 7650 3600
 $Comp
-L basicsensormodule-rescue:TestPoint-Connector TP208
+L Connector:TestPoint TP208
 U 1 1 5AAC8491
 P 8800 3600
@@
 $EndComp
 $Comp
-L basicsensormodule-rescue:TestPoint-Connector TP207
+L Connector:TestPoint TP207
 U 1 1 5AAC8C25
 P 7600 3600
